File: Hardware/PCB Design/KiCAD Files/oBeMs_Pulse_PCB.sch (KiCad schematic (older format))
At the start: 37 parts

Commit message: Update Schematic and add presentation
Parts:
- removed P?: LED, symbol CONN_01X02
- removed P?: 1WIRE_OUT, symbol CONN_01X02
- removed P?: 1WIRE_IN, symbol CONN_01X02
- added C1: 100n, symbol C
- added C2: 0.1u, symbol CP1
- added C3: 10n, symbol CP1
- added C4: 330u, symbol CP1
- added D1: 1N4001, symbol DIODE
- added D10, D5, D6, D7, D8, D9: LED, symbol LED
- added D2: WDT, symbol LED
- added P10: LED, symbol CONN_01X08
- added P12: ADC_VREF_2, symbol CONN_01X02
- added P13: ADC_VREF_1, symbol CONN_01X02
- added P17: DIO_7-12, symbol CONN_01X06
- added P18: DIO_1-6, symbol CONN_01X06
- added P19, P20: PULL_DOWN, symbol CONN_02X06
- added P2: HARD_WDT, symbol CONN_01X04
- added P21: PULL_UP, symbol CONN_02X06
- added P23: DIO_7-12, symbol CONN_01X12
- added P3: 1WIRE_OUT, symbol CONN_01X03
- added P6: 1WIRE_SENSOR, symbol CONN_01X03
- added R1, R2, R6: 10k, symbol R
- added R10, R11, R12, R13, R14, R15, R17, R19, R21, R23, R25, R4, R9: 120, symbol R
- added R5: 390k, symbol R
- added U1: TLC555, symbol TLC555
- P22: renamed from P?; value CONN_02X06 -> PULL_UP
- P24: renamed from P?; value DIO_1_6 -> DIO_1-6
- gave numbers to parts that had none: 32
Connections:
- wire segments 214 -> 407
Other:
- moved on the sheet: CPU1, F1, P1, P11, P14, P16, P24, P4, P5, P7, P8, P9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

Commit message: Update Schematic WDT and PSU
Parts:
- removed C6: 1u, symbol C
- removed U3: MCP1826S-3302, symbol MCP1826S-3302
- added C6: 330u, symbol CP1
- added D11: IN5819, symbol ZENER
- added L1: 330uH, symbol INDUCTOR
- added Q1: NPN, symbol NPN
- added R27, R28: 47k, symbol R
- added R29: 1k, symbol R
- added R30: 10R, symbol R
- added U3: MCP6241, symbol MCP6241
- added U6: LM2575, symbol LM2575
- C5: value 4.7u -> 100u
- R2: value 10k -> 1M
Connections:
- wire segments 407 -> 433
- no-connect marks 3 -> 6
Other:
- moved on the sheet: D1, P2, P3, P6, U1, U2

Commit message: Update to initial version of PCB
Initial PCB version.
Parts:
- removed C1, C7, C8: 100n, symbol C
- removed C2: 0.1u, symbol CP1
- removed C3: 10n, symbol CP1
- removed C4, C6: 330u, symbol CP1
- removed C5: 100u, symbol CP1
- removed D1: 1N4001, symbol DIODE
- removed D10, D3, D4, D5, D6, D7, D8, D9: LED, symbol LED
- removed D11: IN5819, symbol ZENER
- removed D2: WDT, symbol LED
- removed F1: 500mA FUSE, symbol FUSE
- removed L1: 330uH, symbol INDUCTOR
- removed P10: LED, symbol CONN_01X08
- removed P11: 5V, symbol CONN_02X04
- removed P12: ADC_VREF_2, symbol CONN_01X02
- removed P13: ADC_VREF_1, symbol CONN_01X02
- removed P14: 3V3, symbol CONN_02X04
- removed P15: SPI_ADC, symbol CONN_01X07
- removed P16: GND, symbol CONN_02X04
- removed P17: DIO_7-12, symbol CONN_01X06
- removed P18: DIO_1-6, symbol CONN_01X06
- removed P19, P20: PULL_DOWN, symbol CONN_02X06
- removed P21, P22: PULL_UP, symbol CONN_02X06
- removed P23: DIO_7-12, symbol CONN_01X12
- removed P24: DIO_1-6, symbol CONN_01X12
- removed P8: ADC_0-7, symbol CONN_02X08
- removed P9: ADC_8-15, symbol CONN_02X08
- removed PSU1: PSU_10W_5V, symbol PSU_10W_5V
- removed Q1: NPN, symbol NPN
- removed R1, R6: 10k, symbol R
- removed R10, R11, R12, R13, R14, R15, R16, R17, R18, R19, R20, R21, R22, R23, R24, R25, R26, R4, R7, R8, R9: 120, symbol R
- removed R2: 1M, symbol R
- removed R27, R28: 47k, symbol R
- removed R29: 1k, symbol R
- removed R3: 4k7, symbol R
- removed R30: 10R, symbol R
- removed R5: 390k, symbol R
- removed U1: TLC555, symbol TLC555
- removed U2: DS18B20, symbol DS18B20
- removed U3: MCP6241, symbol MCP6241
- removed U4, U5: MCP3008, symbol MCP3008
- removed U6: LM2575, symbol LM2575
- added LG1: REI Logo, matts_components:reinnovation_logo_15mm, symbol CONN_01X01
- added LG3: OSHW Logo, T4Logo:OSHW_13mm, symbol CONN_01X01
- added P4: LED 5-8, REInnovationFootprint:Pin_Header_Straight_1x04, symbol CONN_01X04
- added P5: AC_INPUT_PLUG, Pin_Headers:Pin_Header_Angled_1x03, symbol CONN_01X03
- added P7: LED 1-4, REInnovationFootprint:Pin_Header_Straight_1x04, symbol CONN_01X04
- CPU1: footprint (none) -> REInnovationFootprint:RPi_B_B+_MOUNTING
- LG2: renamed from P5; value Logo -> T4 Logo; footprint (none) -> Logo:T4_32mm
- P1: renamed from P3; footprint (none) -> Pin_Headers:Pin_Header_Straight_1x03
- P2: renamed from P6; footprint (none) -> Pin_Headers:Pin_Header_Straight_1x03
- P3: renamed from P2; footprint (none) -> REInnovationFootprint:TH_4x1_CONN
- P6: renamed from P1; footprint (none) -> REInnovationFootprint:TH_3W_CamdenBoss; Description (none) -> 240V AC >3A; Manufacturer (none) -> CamdenBoss; Manufacturer Part No (none) -> CTB9358/3; Supplier 1 (none) -> CPC; Supplier 1 Part No (none) -> CN11626
- PCB1: renamed from P7; footprint (none) -> REInnovationFootprint:PCB_120x150_WISKA
- renumbered P4 to EN1
Connections:
- net labels removed: +5V, GNDPWR
- wire segments 433 -> 29
- no-connect marks 6 -> 8
Other:
- note removed: "1 Wire Temp Monitoring"
- note removed: "3.3V LDO 1A Regulator"
- note removed: "5V Supply"
- note removed: "DIO"
- note removed: "Distribution Blocks for Power"
- note removed: "Output LED"
- note removed: "SPI ADC 8 Channel"
- note removed: "Watch Dog Timer"
- moved on the sheet: CPU1, EN1, LG2, P1, P2, P3, P6, PCB1

Commit message: Version 3 revision
Added 3A switching 5V supply and Capacitors axial and radial
Parts:
- added P8: VIN_DC, REInnovationFootprint:DC_Power_2_1, symbol BARREL_JACK
- LG2: footprint Logo:T4_32mm -> PCB_logo:T4_32mm
- LG3: footprint T4Logo:OSHW_13mm -> PCB_logo:OSHW_13mm
- P5: footprint Pin_Headers:Pin_Header_Angled_1x03 -> (none)
Connections:
- wire segments 29 -> 33
Changed lines of the file:
@@
 LIBS:contrib
 LIBS:valves
+LIBS:oBeMs_Pulse_PCB-cache
 LIBS:matts_components
-LIBS:oBeMs_Pulse_PCB-cache
 EELAYER 25 0
 EELAYER END
@@
 Title "oBeMs Open Pulse Monitor Unit"
 Date "2015-11-01"
-Rev "2"
+Rev "3"
 Comp "T4 Sustainability"
 Comment1 "PCB design by RE-Innovation"
@@
 F 0 "LG2" H 6100 7100 50  0000 C CNN
 F 1 "T4 Logo" V 6200 7000 50  0000 C CNN
-F 2 "Logo:T4_32mm" H 6100 7000 60  0001 C CNN
+F 2 "PCB_logo:T4_32mm" H 6100 7000 60  0001 C CNN
 F 3 "" H 6100 7000 60  0000 C CNN
 	1    6100 7000
@@
 F 0 "P5" H 1200 1650 50  0000 C CNN
 F 1 "AC_INPUT_PLUG" V 1300 1450 50  0000 C CNN
-F 2 "Pin_Headers:Pin_Header_Angled_1x03" H 1200 1450 60  0001 C CNN
+F 2 "" H 1200 1450 60  0001 C CNN
 F 3 "http://www.farnell.com/datasheets/1826287.pdf" H 1200 1450 60  0001 C CNN
 F 4 "240V AC >3A PLUG" H 1200 1450 60  0001 C CNN "Description"
@@
 F 10 "~" H 1200 1450 60  0001 C CNN "Supplier 2"
 F 11 "~" H 1200 1450 60  0001 C CNN "Supplier 2 Part No"
+F 12 "~" H 1200 1450 60  0001 C CNN "Cost"
 	1    1200 1450
 	1    0    0    1
@@
 NoConn ~ 1000 1550
 $Sheet
-S 1900 1100 750  650
+S 1900 1100 750  1150
 U 563600A1
 F0 "PowerSupply" 60
@@
 F3 "N" I L 1900 1450 60
 F4 "EARTH" I L 1900 1550 60
+F5 "VDC_IN_GND" I L 1900 2100 60
+F6 "VDC_IN+" I L 1900 1950 60
 $EndSheet
 Wire Wire Line
@@
 F 0 "LG3" H 6100 7500 50  0000 C CNN
 F 1 "OSHW Logo" V 6200 7400 50  0000 C CNN
-F 2 "T4Logo:OSHW_13mm" H 6100 7400 60  0001 C CNN
+F 2 "PCB_logo:OSHW_13mm" H 6100 7400 60  0001 C CNN
 F 3 "" H 6100 7400 60  0000 C CNN
 	1    6100 7400
@@
 	-1   0    0    1
 $EndComp
+Wire Wire Line
+	1500 1950 1900 1950
+$Comp
+L BARREL_JACK P8
+U 1 1 5672DA00
+P 1200 2050
+F 0 "P8" H 1200 2300 50  0000 C CNN
+F 1 "VIN_DC" H 1200 1850 50  0000 C CNN
+F 2 "REInnovationFootprint:DC_Power_2_1" H 1200 2050 50  0001 C CNN
+F 3 "" H 1200 2050 50  0000 C CNN
+	1    1200 2050
+	1    0    0    -1
+$EndComp
+Wire Wire Line
+	1500 2150 1750 2150
+Wire Wire Line
+	1750 2150 1750 2100
+Wire Wire Line
+	1750 2100 1900 2100
 $EndSCHEMATC

Commit message: Updated small changes.
Info and changes from email 18/12/15.
Parts:
- removed P8: VIN_DC, REInnovationFootprint:DC_Power_2_1, symbol BARREL_JACK
- added H1, H2: Bolt Hole, REInnovationFootprint:3mm_hole, symbol CONN_01X01
- added P8: VDC_IN, REInnovationFootprint:TH_CONN_2W, symbol CONN_01X02
Connections:
- no-connect marks 8 -> 10
Changed lines of the file:
@@
 Wire Wire Line
 	1500 1950 1900 1950
+Wire Wire Line
+	1750 2100 1900 2100
 $Comp
-L BARREL_JACK P8
-U 1 1 5672DA00
-P 1200 2050
-F 0 "P8" H 1200 2300 50  0000 C CNN
-F 1 "VIN_DC" H 1200 1850 50  0000 C CNN
-F 2 "REInnovationFootprint:DC_Power_2_1" H 1200 2050 50  0001 C CNN
-F 3 "" H 1200 2050 50  0000 C CNN
-	1    1200 2050
+L CONN_01X02 P8
+U 1 1 5675A266
+P 1300 2000
+F 0 "P8" H 1300 2150 50  0000 C CNN
+F 1 "VDC_IN" V 1400 2000 50  0000 C CNN
+F 2 "REInnovationFootprint:TH_CONN_2W" H 1300 2000 50  0001 C CNN
+F 3 "" H 1300 2000 50  0000 C CNN
+F 4 "~" H 1300 2000 60  0001 C CNN "Description"
+F 5 "~" H 1300 2000 60  0001 C CNN "Notes"
+F 6 "~" H 1300 2000 60  0001 C CNN "Manufacturer"
+F 7 "~" H 1300 2000 60  0001 C CNN "Manufacturer Part No"
+F 8 "~" H 1300 2000 60  0001 C CNN "Supplier 1"
+F 9 "~" H 1300 2000 60  0001 C CNN "Supplier 1 Part No"
+F 10 "~" H 1300 2000 60  0001 C CNN "Supplier 2"
+F 11 "~" H 1300 2000 60  0001 C CNN "Supplier 2 Part No"
+F 12 "~" H 1300 2000 60  0001 C CNN "Cost"
+	1    1300 2000
+	-1   0    0    -1
+$EndComp
+Wire Wire Line
+	1500 2050 1750 2050
+Wire Wire Line
+	1750 2050 1750 2100
+$Comp
+L CONN_01X01 H1
+U 1 1 5675BB5B
+P 3200 1550
+F 0 "H1" H 3200 1650 50  0000 C CNN
+F 1 "Bolt Hole" V 3300 1550 50  0000 C CNN
+F 2 "REInnovationFootprint:3mm_hole" H 3200 1550 50  0001 C CNN
+F 3 "" H 3200 1550 50  0000 C CNN
+	1    3200 1550
 	1    0    0    -1
 $EndComp
-Wire Wire Line
-	1500 2150 1750 2150
-Wire Wire Line
-	1750 2150 1750 2100
-Wire Wire Line
-	1750 2100 1900 2100
+$Comp
+L CONN_01X01 H2
+U 1 1 5675BC36
+P 3200 2000
+F 0 "H2" H 3200 2100 50  0000 C CNN
+F 1 "Bolt Hole" V 3300 2000 50  0000 C CNN
+F 2 "REInnovationFootprint:3mm_hole" H 3200 2000 50  0001 C CNN
+F 3 "" H 3200 2000 50  0000 C CNN
+	1    3200 2000
+	1    0    0    -1
+$EndComp
+NoConn ~ 3000 1550
+NoConn ~ 3000 2000
 $EndSCHEMATC

Commit message: Updates from email 21/12/15
Parts:
- removed P1: 1WIRE_OUT, Pin_Headers:Pin_Header_Straight_1x03, symbol CONN_01X03
- removed P2: 1WIRE_SENSOR, Pin_Headers:Pin_Header_Straight_1x03, symbol CONN_01X03
- added LG4: V0000, symbol CONN_01X01
- added P1: 1WIRE, REInnovationFootprint:Pin_Header_Straight_1x04, symbol CONN_01X04
Connections:
- net TemperatureSensor/+3.3V: now also P1.1 (P1)
- net TemperatureSensor/D-1-Wire: now also P1.2 (P2), P1.3 (P3)
- net TemperatureSensor/GND: now also P1.4 (P4)
- net PowerSupply/VDC_IN+ renamed PowerSupply/VIN_A
- net PowerSupply/VDC_IN_GND renamed PowerSupply/VIN_B
- no-connect marks 10 -> 11
Other:
- note added: "VERSION NUMBER"
Changed lines of the file:
@@
 LIBS:contrib
 LIBS:valves
+LIBS:matts_components
 LIBS:oBeMs_Pulse_PCB-cache
-LIBS:matts_components
 EELAYER 25 0
 EELAYER END
@@
 Sheet 1 10
 Title "oBeMs Open Pulse Monitor Unit"
-Date "2015-11-01"
-Rev "3"
+Date "2015-12-21"
+Rev "4"
 Comp "T4 Sustainability"
 Comment1 "PCB design by RE-Innovation"
@@
 	1    7150 2150
 	1    0    0    -1
-$EndComp
-$Comp
-L CONN_01X03 P1
-U 1 1 561517E1
-P 1100 3050
-F 0 "P1" H 1100 3250 50  0000 C CNN
-F 1 "1WIRE_OUT" V 1200 3050 50  0000 C CNN
-F 2 "Pin_Headers:Pin_Header_Straight_1x03" H 1100 3050 60  0001 C CNN
-F 3 "" H 1100 3050 60  0000 C CNN
-	1    1100 3050
-	-1   0    0    -1
-$EndComp
-$Comp
-L CONN_01X03 P2
-U 1 1 56151894
-P 1100 3600
-F 0 "P2" H 1100 3800 50  0000 C CNN
-F 1 "1WIRE_SENSOR" V 1200 3600 50  0000 C CNN
-F 2 "Pin_Headers:Pin_Header_Straight_1x03" H 1100 3600 60  0001 C CNN
-F 3 "" H 1100 3600 60  0000 C CNN
-	1    1100 3600
-	-1   0    0    -1
 $EndComp
 $Comp
@@
 F3 "N" I L 1900 1450 60
 F4 "EARTH" I L 1900 1550 60
-F5 "VDC_IN_GND" I L 1900 2100 60
-F6 "VDC_IN+" I L 1900 1950 60
+F5 "VIN_B" I L 1900 2100 60
+F6 "VIN_A" I L 1900 1950 60
 $EndSheet
 Wire Wire Line
@@
 $EndSheet
 Wire Wire Line
-	1650 3500 1300 3500
-Wire Wire Line
-	1650 2950 1650 3500
-Wire Wire Line
-	1650 2950 1300 2950
-Wire Wire Line
-	1300 3050 1600 3050
-Wire Wire Line
-	1600 3050 1600 3600
-Wire Wire Line
-	1600 3600 1300 3600
-Wire Wire Line
-	1300 3150 1550 3150
-Wire Wire Line
-	1550 3150 1550 3700
-Wire Wire Line
-	1550 3700 1300 3700
-Wire Wire Line
 	1550 3400 1850 3400
-Connection ~ 1550 3400
-Wire Wire Line
-	1850 3300 1600 3300
-Connection ~ 1600 3300
-Wire Wire Line
-	1850 3200 1650 3200
-Connection ~ 1650 3200
+Wire Wire Line
+	1350 3300 1850 3300
+Wire Wire Line
+	1350 3200 1850 3200
 $Sheet
 S 1650 4850 800  600
@@
 NoConn ~ 3000 1550
 NoConn ~ 3000 2000
+$Comp
+L CONN_01X01 LG4
+U 1 1 5677EAF3
+P 4750 7050
+F 0 "LG4" H 4750 7150 50  0000 C CNN
+F 1 "V0000" V 4850 7050 50  0000 C CNN
+F 2 "" H 4750 7050 60  0001 C CNN
+F 3 "" H 4750 7050 60  0000 C CNN
+F 4 "Value" H 4750 7050 60  0001 C CNN "Description"
+F 5 "Value" H 4750 7050 60  0001 C CNN "Notes"
+F 6 "Value" H 4750 7050 60  0001 C CNN "Manufacturer"
+F 7 "Value" H 4750 7050 60  0001 C CNN "Manufacturer Part No"
+F 8 "Value" H 4750 7050 60  0001 C CNN "Supplier 1"
+F 9 "Value" H 4750 7050 60  0001 C CNN "Supplier 1 Part No"
+F 10 "Value" H 4750 7050 60  0001 C CNN "Supplier 2"
+F 11 "Value" H 4750 7050 60  0001 C CNN "Supplier 2 Part No"
+	1    4750 7050
+	1    0    0    -1
+$EndComp
+NoConn ~ 4550 7050
+Text Notes 4300 6850 0    60   ~ 0
+VERSION NUMBER
+$Comp
+L CONN_01X04 P1
+U 1 1 56780130
+P 1150 3350
+F 0 "P1" H 1150 3600 50  0000 C CNN
+F 1 "1WIRE" V 1250 3350 50  0000 C CNN
+F 2 "REInnovationFootprint:Pin_Header_Straight_1x04" H 1150 3350 60  0001 C CNN
+F 3 "" H 1150 3350 60  0000 C CNN
+	1    1150 3350
+	-1   0    0    -1
+$EndComp
+Wire Wire Line
+	1350 3500 1550 3500
+Wire Wire Line
+	1550 3500 1550 3400
+Wire Wire Line
+	1350 3400 1400 3400
+Wire Wire Line
+	1400 3400 1400 3300
+Connection ~ 1400 3300
 $EndSCHEMATC

Commit message: More small changes 22/12/15
Parts:
- P8: value VDC_IN -> LT_PWR
Changed lines of the file:
@@
 LIBS:contrib
 LIBS:valves
+LIBS:oBeMs_Pulse_PCB-cache
 LIBS:matts_components
-LIBS:oBeMs_Pulse_PCB-cache
 EELAYER 25 0
 EELAYER END
@@
 Sheet 1 10
 Title "oBeMs Open Pulse Monitor Unit"
-Date "2015-12-21"
-Rev "4"
+Date "2015-12-22"
+Rev "5"
 Comp "T4 Sustainability"
 Comment1 "PCB design by RE-Innovation"
@@
 P 1300 2000
 F 0 "P8" H 1300 2150 50  0000 C CNN
-F 1 "VDC_IN" V 1400 2000 50  0000 C CNN
+F 1 "LT_PWR" V 1400 2000 50  0000 C CNN
 F 2 "REInnovationFootprint:TH_CONN_2W" H 1300 2000 50  0001 C CNN
 F 3 "" H 1300 2000 50  0000 C CNN

Commit message: Rev 6. Final changes before PCB v0000 done
Parts:
- H1, H2: value Bolt Hole -> AC Cover Mount Hole
Connections:
- net TemperatureSensor/+3.3V is gone; now on net +3.3V: P1.1 (P1)
- net TemperatureSensor/GND is gone; now on net GND: P1.4 (P4)
Other:
- moved on the sheet: H1, H2
