File: Hardware/PCB Design/KiCAD Files/oBeMs_Pulse_PCB.sch (KiCad schematic (older format))
At the start: 16 parts, among them P1 1WIRE, P3 HARD_WDT, P4 LED 5-8, P5 AC_INPUT_PLUG, P6 AC_INPUT, P7 LED 1-4, P8 LT_PWR

Commit message: Changes for v0001
Multiple PCb changes. 50Pcs ordered
Parts:
- added R10: 1M, REInnovationFootprint:TH_Resistor_1, symbol R
- P8: footprint REInnovationFootprint:TH_CONN_2W -> REInnovationFootprint:TH_CONN_2W_LGPAD
Connections:
- wire segments 51 -> 55
Changed lines of the file:
@@
 EESchema Schematic File Version 2
-LIBS:oBeMs_Pulse_PCB-rescue
 LIBS:power
 LIBS:device
@@
 F 0 "P8" H 1300 2150 50  0000 C CNN
 F 1 "LT_PWR" V 1400 2000 50  0000 C CNN
-F 2 "REInnovationFootprint:TH_CONN_2W" H 1300 2000 50  0001 C CNN
+F 2 "REInnovationFootprint:TH_CONN_2W_LGPAD" H 1300 2000 50  0001 C CNN
 F 3 "" H 1300 2000 50  0000 C CNN
 F 4 "~" H 1300 2000 60  0001 C CNN "Description"
@@
 Connection ~ 8750 1300
 $Comp
-L GND-RESCUE-oBeMs_Pulse_PCB #PWR?
+L GND-RESCUE-oBeMs_Pulse_PCB #PWR013
 U 1 1 567BE5A0
 P 2950 1950
-F 0 "#PWR?" H 2950 1950 30  0001 C CNN
+F 0 "#PWR013" H 2950 1950 30  0001 C CNN
 F 1 "GND" H 2950 1880 30  0001 C CNN
 F 2 "" H 2950 1950 60  0000 C CNN
@@
 $EndComp
 $Comp
-L +3.3V-RESCUE-oBeMs_Pulse_PCB #PWR?
+L +3.3V-RESCUE-oBeMs_Pulse_PCB #PWR014
 U 1 1 567BE5A7
 P 3100 1700
-F 0 "#PWR?" H 3100 1660 30  0001 C CNN
+F 0 "#PWR014" H 3100 1660 30  0001 C CNN
 F 1 "+3.3V" H 3100 1810 30  0000 C CNN
 F 2 "" H 3100 1700 60  0000 C CNN
@@
 $EndComp
 $Comp
-L +5V #PWR?
+L +5V #PWR015
 U 1 1 567BE5AD
 P 2950 1450
-F 0 "#PWR?" H 2950 1540 20  0001 C CNN
+F 0 "#PWR015" H 2950 1540 20  0001 C CNN
 F 1 "+5V" H 2950 1600 30  0000 C CNN
 F 2 "" H 2950 1450 60  0000 C CNN
@@
 Wire Wire Line
 	2950 1900 2950 1950
+$Comp
+L R R10
+U 1 1 5991A267
+P 2250 2500
+F 0 "R10" V 2330 2500 50  0000 C CNN
+F 1 "1M" V 2250 2500 50  0000 C CNN
+F 2 "REInnovationFootprint:TH_Resistor_1" V 2180 2500 50  0001 C CNN
+F 3 "" H 2250 2500 50  0000 C CNN
+	1    2250 2500
+	0    1    1    0
+$EndComp
+Wire Wire Line
+	2100 2500 1800 2500
+Wire Wire Line
+	1800 2500 1800 1550
+Connection ~ 1800 1550
+Wire Wire Line
+	2800 1900 2800 2500
+Wire Wire Line
+	2800 2500 2400 2500
+Connection ~ 2800 1900
 $EndSCHEMATC
