File: Hardware/PCB Design/KiCAD Files/ADC_DAC.sch (KiCad schematic (older format))
At the start: 13 parts, among them P13 ADC_0-7, P14 ADC_8-15, P15 ADC_VREF_2, P16 ADC_VREF_1, P17 SPI_ADC_DAC, P34 DAC_A, P35 DAC_B, U5 MCP3008, U6 MCP3008, U7 MCP4802

Commit message: Version 3 revision
Added 3A switching 5V supply and Capacitors axial and radial
Parts:
- P13, P14: footprint Pin_Headers:Pin_Header_Straight_2x08 -> REInnovationFootprint:Pin_Header_Straight_2x08
- P15, P16, P34, P35: footprint Pin_Headers:Pin_Header_Straight_1x02 -> REInnovationFootprint:Pin_Header_Straight_1x02
- P17: footprint Pin_Headers:Pin_Header_Straight_1x08 -> REInnovationFootprint:Pin_Header_Straight_1x08
Changed lines of the file:
@@
 LIBS:contrib
 LIBS:valves
+LIBS:oBeMs_Pulse_PCB-cache
 LIBS:matts_components
-LIBS:oBeMs_Pulse_PCB-cache
 EELAYER 25 0
 EELAYER END
@@
 Title "oBeMs Open Pulse Monitor Unit"
 Date "2015-11-01"
-Rev "2"
+Rev "3"
 Comp "T4 Sustainability"
 Comment1 "PCB design by RE-Innovation"
@@
 F 0 "P13" H 3950 3300 50  0000 C CNN
 F 1 "ADC_0-7" V 3950 2850 50  0000 C CNN
-F 2 "Pin_Headers:Pin_Header_Straight_2x08" H 3950 1650 60  0001 C CNN
+F 2 "REInnovationFootprint:Pin_Header_Straight_2x08" H 3950 1650 60  0001 C CNN
 F 3 "" H 3950 1650 60  0000 C CNN
 	1    3950 2850
@@
 $EndComp
 $Comp
-L GND-RESCUE-oBeMs_Pulse_PCB #PWR016
+L GND-RESCUE-oBeMs_Pulse_PCB #PWR018
 U 1 1 563769DC
 P 5450 3250
-F 0 "#PWR016" H 5450 3250 30  0001 C CNN
+F 0 "#PWR018" H 5450 3250 30  0001 C CNN
 F 1 "GND" H 5450 3180 30  0001 C CNN
 F 2 "" H 5450 3250 60  0000 C CNN
@@
 $EndComp
 $Comp
-L +3.3V-RESCUE-oBeMs_Pulse_PCB #PWR017
+L +3.3V-RESCUE-oBeMs_Pulse_PCB #PWR019
 U 1 1 563769E2
 P 5450 2450
-F 0 "#PWR017" H 5450 2410 30  0001 C CNN
+F 0 "#PWR019" H 5450 2410 30  0001 C CNN
 F 1 "+3.3V" H 5450 2560 30  0000 C CNN
 F 2 "" H 5450 2450 60  0000 C CNN
@@
 $EndComp
 $Comp
-L GND-RESCUE-oBeMs_Pulse_PCB #PWR018
+L GND-RESCUE-oBeMs_Pulse_PCB #PWR020
 U 1 1 563769EF
 P 7450 3450
-F 0 "#PWR018" H 7450 3450 30  0001 C CNN
+F 0 "#PWR020" H 7450 3450 30  0001 C CNN
 F 1 "GND" H 7450 3380 30  0001 C CNN
 F 2 "" H 7450 3450 60  0000 C CNN
@@
 $EndComp
 $Comp
-L +3.3V-RESCUE-oBeMs_Pulse_PCB #PWR019
+L +3.3V-RESCUE-oBeMs_Pulse_PCB #PWR021
 U 1 1 563769F5
 P 7450 2700
-F 0 "#PWR019" H 7450 2660 30  0001 C CNN
+F 0 "#PWR021" H 7450 2660 30  0001 C CNN
 F 1 "+3.3V" H 7450 2810 30  0000 C CNN
 F 2 "" H 7450 2700 60  0000 C CNN
@@
 F 0 "P14" H 3950 4550 50  0000 C CNN
 F 1 "ADC_8-15" V 3950 4100 50  0000 C CNN
-F 2 "Pin_Headers:Pin_Header_Straight_2x08" H 3950 2900 60  0001 C CNN
+F 2 "REInnovationFootprint:Pin_Header_Straight_2x08" H 3950 2900 60  0001 C CNN
 F 3 "" H 3950 2900 60  0000 C CNN
 	1    3950 4100
@@
 $EndComp
 $Comp
-L GND-RESCUE-oBeMs_Pulse_PCB #PWR020
+L GND-RESCUE-oBeMs_Pulse_PCB #PWR022
 U 1 1 56376A18
 P 5450 4500
-F 0 "#PWR020" H 5450 4500 30  0001 C CNN
+F 0 "#PWR022" H 5450 4500 30  0001 C CNN
 F 1 "GND" H 5450 4430 30  0001 C CNN
 F 2 "" H 5450 4500 60  0000 C CNN
@@
 $EndComp
 $Comp
-L +3.3V-RESCUE-oBeMs_Pulse_PCB #PWR021
+L +3.3V-RESCUE-oBeMs_Pulse_PCB #PWR023
 U 1 1 56376A1E
 P 5450 3700
-F 0 "#PWR021" H 5450 3660 30  0001 C CNN
+F 0 "#PWR023" H 5450 3660 30  0001 C CNN
 F 1 "+3.3V" H 5450 3810 30  0000 C CNN
 F 2 "" H 5450 3700 60  0000 C CNN
@@
 F 0 "P16" H 6500 2650 50  0000 C CNN
 F 1 "ADC_VREF_1" V 6650 2500 50  0000 C CNN
-F 2 "Pin_Headers:Pin_Header_Straight_1x02" H 6500 2500 60  0001 C CNN
+F 2 "REInnovationFootprint:Pin_Header_Straight_1x02" H 6500 2500 60  0001 C CNN
 F 3 "" H 6500 2500 60  0000 C CNN
 	1    6500 2500
@@
 F 0 "P15" H 6350 3950 50  0000 C CNN
 F 1 "ADC_VREF_2" V 6450 3800 50  0000 C CNN
-F 2 "Pin_Headers:Pin_Header_Straight_1x02" H 6350 3800 60  0001 C CNN
+F 2 "REInnovationFootprint:Pin_Header_Straight_1x02" H 6350 3800 60  0001 C CNN
 F 3 "" H 6350 3800 60  0000 C CNN
 	1    6350 3800
@@
 $EndComp
 $Comp
-L GND-RESCUE-oBeMs_Pulse_PCB #PWR022
+L GND-RESCUE-oBeMs_Pulse_PCB #PWR024
 U 1 1 56376A41
 P 6050 2450
-F 0 "#PWR022" H 6050 2450 30  0001 C CNN
+F 0 "#PWR024" H 6050 2450 30  0001 C CNN
 F 1 "GND" H 6050 2380 30  0001 C CNN
 F 2 "" H 6050 2450 60  0000 C CNN
@@
 $EndComp
 $Comp
-L GND-RESCUE-oBeMs_Pulse_PCB #PWR023
+L GND-RESCUE-oBeMs_Pulse_PCB #PWR025
 U 1 1 56376A47
 P 6000 3650
-F 0 "#PWR023" H 6000 3650 30  0001 C CNN
+F 0 "#PWR025" H 6000 3650 30  0001 C CNN
 F 1 "GND" H 6000 3580 30  0001 C CNN
 F 2 "" H 6000 3650 60  0000 C CNN
@@
 F 0 "P17" H 7750 3500 50  0000 C CNN
 F 1 "SPI_ADC_DAC" V 7850 3050 50  0000 C CNN
-F 2 "Pin_Headers:Pin_Header_Straight_1x08" H 7750 3050 60  0001 C CNN
+F 2 "REInnovationFootprint:Pin_Header_Straight_1x08" H 7750 3050 60  0001 C CNN
 F 3 "" H 7750 3050 60  0000 C CNN
 	1    7750 3050
@@
 Connection ~ 6550 4050
 $Comp
-L +3.3V-RESCUE-oBeMs_Pulse_PCB #PWR024
+L +3.3V-RESCUE-oBeMs_Pulse_PCB #PWR026
 U 1 1 563860F4
 P 7300 5200
-F 0 "#PWR024" H 7300 5160 30  0001 C CNN
+F 0 "#PWR026" H 7300 5160 30  0001 C CNN
 F 1 "+3.3V" H 7300 5310 30  0000 C CNN
 F 2 "" H 7300 5200 60  0000 C CNN
@@
 $EndComp
 $Comp
-L GND-RESCUE-oBeMs_Pulse_PCB #PWR025
+L GND-RESCUE-oBeMs_Pulse_PCB #PWR027
 U 1 1 5638611D
 P 8400 5550
-F 0 "#PWR025" H 8400 5550 30  0001 C CNN
+F 0 "#PWR027" H 8400 5550 30  0001 C CNN
 F 1 "GND" H 8400 5480 30  0001 C CNN
 F 2 "" H 8400 5550 60  0000 C CNN
@@
 F 0 "P34" H 8750 5350 50  0000 C CNN
 F 1 "DAC_A" V 8850 5200 50  0000 C CNN
-F 2 "Pin_Headers:Pin_Header_Straight_1x02" H 8750 5200 60  0001 C CNN
+F 2 "REInnovationFootprint:Pin_Header_Straight_1x02" H 8750 5200 60  0001 C CNN
 F 3 "" H 8750 5200 60  0000 C CNN
 	1    8750 5200
@@
 F 0 "P35" H 8750 5950 50  0000 C CNN
 F 1 "DAC_B" V 8850 5800 50  0000 C CNN
-F 2 "Pin_Headers:Pin_Header_Straight_1x02" H 8750 5800 60  0001 C CNN
+F 2 "REInnovationFootprint:Pin_Header_Straight_1x02" H 8750 5800 60  0001 C CNN
 F 3 "" H 8750 5800 60  0000 C CNN
 	1    8750 5800
@@
 Connection ~ 8500 5250
 $Comp
-L GND-RESCUE-oBeMs_Pulse_PCB #PWR026
+L GND-RESCUE-oBeMs_Pulse_PCB #PWR028
 U 1 1 56386BF5
 P 8150 5800
-F 0 "#PWR026" H 8150 5800 30  0001 C CNN
+F 0 "#PWR028" H 8150 5800 30  0001 C CNN
 F 1 "GND" H 8150 5730 30  0001 C CNN
 F 2 "" H 8150 5800 60  0000 C CNN

Commit message: Updates from email 21/12/15
Parts:
- removed P34: DAC_A, REInnovationFootprint:Pin_Header_Straight_1x02, symbol CONN_01X02
- removed P35: DAC_B, REInnovationFootprint:Pin_Header_Straight_1x02, symbol CONN_01X02
- added P34: DAC, REInnovationFootprint:Pin_Header_Straight_2x04, symbol CONN_02X04
- C7, C8: value 100n -> 1000n
Connections:
- net GND: now also P34.2 (P2), P34.4 (P4), P34.6 (P6), P34.8 (P8)
- net at U7.6 (VoutB): now also P34.5 (P5), P34.7 (P7)
- net at U7.8 (VoutA): now also P34.1 (P1), P34.3 (P3)
Changed lines of the file:
@@
 LIBS:contrib
 LIBS:valves
+LIBS:matts_components
 LIBS:oBeMs_Pulse_PCB-cache
-LIBS:matts_components
 EELAYER 25 0
 EELAYER END
@@
 Sheet 6 10
 Title "oBeMs Open Pulse Monitor Unit"
-Date "2015-11-01"
-Rev "3"
+Date "2015-12-21"
+Rev "4"
 Comp "T4 Sustainability"
 Comment1 "PCB design by RE-Innovation"
@@
 P 6050 2200
 F 0 "C8" H 6100 2300 50  0000 L CNN
-F 1 "100n" H 6100 2100 50  0000 L CNN
+F 1 "1000n" H 6100 2100 50  0000 L CNN
 F 2 "matts_components:C1_wide_lg_pad_2" H 6050 2200 60  0001 C CNN
 F 3 "" H 6050 2200 60  0000 C CNN
@@
 P 6000 3400
 F 0 "C7" H 6050 3500 50  0000 L CNN
-F 1 "100n" H 6050 3300 50  0000 L CNN
+F 1 "1000n" H 6050 3300 50  0000 L CNN
 F 2 "matts_components:C1_wide_lg_pad_2" H 6000 3400 60  0001 C CNN
 F 3 "" H 6000 3400 60  0000 C CNN
@@
 Wire Wire Line
 	7300 5400 7300 5200
-$Comp
-L CONN_01X02 P34
-U 1 1 5638622A
-P 8750 5200
-F 0 "P34" H 8750 5350 50  0000 C CNN
-F 1 "DAC_A" V 8850 5200 50  0000 C CNN
-F 2 "REInnovationFootprint:Pin_Header_Straight_1x02" H 8750 5200 60  0001 C CNN
-F 3 "" H 8750 5200 60  0000 C CNN
-	1    8750 5200
-	1    0    0    -1
-$EndComp
-$Comp
-L CONN_01X02 P35
-U 1 1 5638632F
-P 8750 5800
-F 0 "P35" H 8750 5950 50  0000 C CNN
-F 1 "DAC_B" V 8850 5800 50  0000 C CNN
-F 2 "REInnovationFootprint:Pin_Header_Straight_1x02" H 8750 5800 60  0001 C CNN
-F 3 "" H 8750 5800 60  0000 C CNN
-	1    8750 5800
-	1    0    0    -1
-$EndComp
-Wire Wire Line
-	8550 5250 8500 5250
-Wire Wire Line
-	8500 5150 8500 5400
-Wire Wire Line
-	8500 5150 8550 5150
-Wire Wire Line
-	8300 5750 8550 5750
-Wire Wire Line
-	8500 5750 8500 5850
-Wire Wire Line
-	8500 5850 8550 5850
 Wire Wire Line
 	8050 5600 8300 5600
 Wire Wire Line
 	8300 5600 8300 5750
-Connection ~ 8500 5750
-Wire Wire Line
-	8500 5400 8050 5400
-Connection ~ 8500 5250
+Wire Wire Line
+	8050 5400 9200 5400
 $Comp
 L GND-RESCUE-oBeMs_Pulse_PCB #PWR028
@@
 	8200 5200 8200 5500
 Connection ~ 8200 5500
+$Comp
+L CONN_02X04 P34
+U 1 1 5678A781
+P 9450 5450
+F 0 "P34" H 9450 5700 50  0000 C CNN
+F 1 "DAC" H 9450 5200 50  0000 C CNN
+F 2 "REInnovationFootprint:Pin_Header_Straight_2x04" H 9450 4250 60  0001 C CNN
+F 3 "" H 9450 4250 60  0000 C CNN
+	1    9450 5450
+	1    0    0    -1
+$EndComp
+$Comp
+L GND-RESCUE-oBeMs_Pulse_PCB #PWR029
+U 1 1 5678A7D6
+P 9850 5700
+F 0 "#PWR029" H 9850 5700 30  0001 C CNN
+F 1 "GND" H 9850 5630 30  0001 C CNN
+F 2 "" H 9850 5700 60  0000 C CNN
+F 3 "" H 9850 5700 60  0000 C CNN
+	1    9850 5700
+	1    0    0    -1
+$EndComp
+Wire Wire Line
+	9700 5300 9850 5300
+Wire Wire Line
+	9850 5300 9850 5700
+Wire Wire Line
+	9700 5600 9850 5600
+Connection ~ 9850 5600
+Wire Wire Line
+	9700 5500 9850 5500
+Connection ~ 9850 5500
+Wire Wire Line
+	9700 5400 9850 5400
+Connection ~ 9850 5400
+Wire Wire Line
+	9200 5300 9100 5300
+Wire Wire Line
+	9100 5300 9100 5400
+Connection ~ 9100 5400
+Wire Wire Line
+	8300 5750 9100 5750
+Wire Wire Line
+	9100 5750 9100 5500
+Wire Wire Line
+	9100 5500 9200 5500
+Wire Wire Line
+	9200 5600 9100 5600
+Connection ~ 9100 5600
 $EndSCHEMATC

Commit message: Rev 6. Final changes before PCB v0000 done
Connections:
- net +3.3V renamed +3V3
Changed lines of the file:
@@
 encoding utf-8
 Sheet 6 10
-Title "oBeMs Open Pulse Monitor Unit"
-Date "2015-12-22"
-Rev "5"
+Title "oBeMS Open Interface Board 0001"
+Date "2015-12-23"
+Rev "6"
 Comp "T4 Sustainability"
-Comment1 "PCB design by RE-Innovation"
+Comment1 "PCB design by T4 Sustainability/RE-Innovation"
 Comment2 ""
 Comment3 ""
@@
 F 3 "" H 3950 1650 60  0000 C CNN
 	1    3950 2850
-	1    0    0    -1
-$EndComp
-$Comp
-L GND-RESCUE-oBeMs_Pulse_PCB #PWR018
-U 1 1 563769DC
-P 5450 3250
-F 0 "#PWR018" H 5450 3250 30  0001 C CNN
-F 1 "GND" H 5450 3180 30  0001 C CNN
-F 2 "" H 5450 3250 60  0000 C CNN
-F 3 "" H 5450 3250 60  0000 C CNN
-	1    5450 3250
-	1    0    0    -1
-$EndComp
-$Comp
-L +3.3V-RESCUE-oBeMs_Pulse_PCB #PWR019
-U 1 1 563769E2
-P 5450 2450
-F 0 "#PWR019" H 5450 2410 30  0001 C CNN
-F 1 "+3.3V" H 5450 2560 30  0000 C CNN
-F 2 "" H 5450 2450 60  0000 C CNN
-F 3 "" H 5450 2450 60  0000 C CNN
-	1    5450 2450
-	1    0    0    -1
-$EndComp
-$Comp
-L GND-RESCUE-oBeMs_Pulse_PCB #PWR020
-U 1 1 563769EF
-P 7450 3450
-F 0 "#PWR020" H 7450 3450 30  0001 C CNN
-F 1 "GND" H 7450 3380 30  0001 C CNN
-F 2 "" H 7450 3450 60  0000 C CNN
-F 3 "" H 7450 3450 60  0000 C CNN
-	1    7450 3450
-	1    0    0    -1
-$EndComp
-$Comp
-L +3.3V-RESCUE-oBeMs_Pulse_PCB #PWR021
-U 1 1 563769F5
-P 7450 2700
-F 0 "#PWR021" H 7450 2660 30  0001 C CNN
-F 1 "+3.3V" H 7450 2810 30  0000 C CNN
-F 2 "" H 7450 2700 60  0000 C CNN
-F 3 "" H 7450 2700 60  0000 C CNN
-	1    7450 2700
 	1    0    0    -1
 $EndComp
@@
 $EndComp
 $Comp
-L GND-RESCUE-oBeMs_Pulse_PCB #PWR022
-U 1 1 56376A18
-P 5450 4500
-F 0 "#PWR022" H 5450 4500 30  0001 C CNN
-F 1 "GND" H 5450 4430 30  0001 C CNN
-F 2 "" H 5450 4500 60  0000 C CNN
-F 3 "" H 5450 4500 60  0000 C CNN
-	1    5450 4500
-	1    0    0    -1
-$EndComp
-$Comp
-L +3.3V-RESCUE-oBeMs_Pulse_PCB #PWR023
-U 1 1 56376A1E
-P 5450 3700
-F 0 "#PWR023" H 5450 3660 30  0001 C CNN
-F 1 "+3.3V" H 5450 3810 30  0000 C CNN
-F 2 "" H 5450 3700 60  0000 C CNN
-F 3 "" H 5450 3700 60  0000 C CNN
-	1    5450 3700
-	1    0    0    -1
-$EndComp
-$Comp
 L C-RESCUE-oBeMs_Pulse_PCB C7
 U 1 1 56376A2C
@@
 F 3 "" H 6350 3800 60  0000 C CNN
 	1    6350 3800
-	1    0    0    -1
-$EndComp
-$Comp
-L GND-RESCUE-oBeMs_Pulse_PCB #PWR024
-U 1 1 56376A41
-P 6050 2450
-F 0 "#PWR024" H 6050 2450 30  0001 C CNN
-F 1 "GND" H 6050 2380 30  0001 C CNN
-F 2 "" H 6050 2450 60  0000 C CNN
-F 3 "" H 6050 2450 60  0000 C CNN
-	1    6050 2450
-	1    0    0    -1
-$EndComp
-$Comp
-L GND-RESCUE-oBeMs_Pulse_PCB #PWR025
-U 1 1 56376A47
-P 6000 3650
-F 0 "#PWR025" H 6000 3650 30  0001 C CNN
-F 1 "GND" H 6000 3580 30  0001 C CNN
-F 2 "" H 6000 3650 60  0000 C CNN
-F 3 "" H 6000 3650 60  0000 C CNN
-	1    6000 3650
 	1    0    0    -1
 $EndComp
@@
 Connection ~ 3500 2500
 Wire Wire Line
-	7550 2700 7450 2700
+	7300 2700 7550 2700
 Wire Wire Line
 	7550 3400 7450 3400
-Wire Wire Line
-	7450 3400 7450 3450
 Wire Wire Line
 	5350 2600 5700 2600
@@
 Connection ~ 3500 3750
 Wire Wire Line
-	5450 4450 5450 4500
-Wire Wire Line
 	5350 3850 6150 3850
 Wire Wire Line
@@
 	5350 3200 5450 3200
 Wire Wire Line
-	5450 3200 5450 3250
-Wire Wire Line
 	5800 2000 6050 2000
 Wire Wire Line
 	6050 2400 6050 2450
 Wire Wire Line
-	5450 2450 5450 2500
+	5450 2300 5450 2500
 Connection ~ 5450 2500
 Wire Wire Line
@@
 	6000 3650 6000 3600
 Wire Wire Line
-	5450 3700 5450 3750
+	5450 3550 5450 3750
 Connection ~ 5450 3750
 Connection ~ 5800 3750
@@
 	6550 5600 7300 5600
 Connection ~ 6550 4050
-$Comp
-L +3.3V-RESCUE-oBeMs_Pulse_PCB #PWR026
-U 1 1 563860F4
-P 7300 5200
-F 0 "#PWR026" H 7300 5160 30  0001 C CNN
-F 1 "+3.3V" H 7300 5310 30  0000 C CNN
-F 2 "" H 7300 5200 60  0000 C CNN
-F 3 "" H 7300 5200 60  0000 C CNN
-	1    7300 5200
-	1    0    0    -1
-$EndComp
-$Comp
-L GND-RESCUE-oBeMs_Pulse_PCB #PWR027
-U 1 1 5638611D
-P 8400 5550
-F 0 "#PWR027" H 8400 5550 30  0001 C CNN
-F 1 "GND" H 8400 5480 30  0001 C CNN
-F 2 "" H 8400 5550 60  0000 C CNN
-F 3 "" H 8400 5550 60  0000 C CNN
-	1    8400 5550
-	1    0    0    -1
-$EndComp
 Wire Wire Line
 	8050 5500 8400 5500
@@
 	8400 5500 8400 5550
 Wire Wire Line
-	7300 5400 7300 5200
+	7300 5000 7300 5400
 Wire Wire Line
 	8050 5600 8300 5600
@@
 Wire Wire Line
 	8050 5400 9200 5400
-$Comp
-L GND-RESCUE-oBeMs_Pulse_PCB #PWR028
-U 1 1 56386BF5
-P 8150 5800
-F 0 "#PWR028" H 8150 5800 30  0001 C CNN
-F 1 "GND" H 8150 5730 30  0001 C CNN
-F 2 "" H 8150 5800 60  0000 C CNN
-F 3 "" H 8150 5800 60  0000 C CNN
-	1    8150 5800
-	1    0    0    -1
-$EndComp
 Wire Wire Line
 	8050 5700 8150 5700
@@
 	1    0    0    -1
 $EndComp
-$Comp
-L GND-RESCUE-oBeMs_Pulse_PCB #PWR029
-U 1 1 5678A7D6
-P 9850 5700
-F 0 "#PWR029" H 9850 5700 30  0001 C CNN
-F 1 "GND" H 9850 5630 30  0001 C CNN
-F 2 "" H 9850 5700 60  0000 C CNN
-F 3 "" H 9850 5700 60  0000 C CNN
-	1    9850 5700
-	1    0    0    -1
-$EndComp
 Wire Wire Line
 	9700 5300 9850 5300
 Wire Wire Line
-	9850 5300 9850 5700
+	9850 5300 9850 5750
 Wire Wire Line
 	9700 5600 9850 5600
@@
 	9200 5600 9100 5600
 Connection ~ 9100 5600
+Text HLabel 7450 3400 0    60   Input ~ 0
+GND
+Text HLabel 7300 2700 0    60   Input ~ 0
++3V3
+Text HLabel 5300 3550 0    60   Input ~ 0
++3V3
+Text HLabel 5300 2300 0    60   Input ~ 0
++3V3
+Text HLabel 7300 5000 1    60   Input ~ 0
++3V3
+Wire Wire Line
+	5300 3550 5450 3550
+Wire Wire Line
+	5300 2300 5450 2300
+Text HLabel 6050 2450 0    60   Input ~ 0
+GND
+Text HLabel 5450 3200 2    60   Input ~ 0
+GND
+Text HLabel 6000 3650 0    60   Input ~ 0
+GND
+Text HLabel 5450 4450 2    60   Input ~ 0
+GND
+Text HLabel 8400 5550 2    60   Input ~ 0
+GND
+Text HLabel 8150 5800 3    60   Input ~ 0
+GND
+Text HLabel 9850 5750 3    60   Input ~ 0
+GND
 $EndSCHEMATC

Commit message: Changes for v0001
Multiple PCb changes. 50Pcs ordered
Parts:
- removed U5, U6: MCP3008, REInnovationFootprint:DIP-16__300_ELL_lg_pad, symbol MCP3008
- added R55, R56, R57: 100k, REInnovationFootprint:TH_Resistor_1, symbol R
- added U5, U6: MCP3008, REInnovationFootprint:DIP-16__300_ELL_lg_pad, symbol MCP3008_16pin
- C7, C8: value 1000n -> 1u
- C9: value 100n -> 1u
- U7: value MCP4802 -> MCP4812
Connections:
- wire segments 108 -> 123
Other:
- note added: "~CS~ PULL UP"
Changed lines of the file:
@@
 EESchema Schematic File Version 2
-LIBS:oBeMs_Pulse_PCB-rescue
 LIBS:power
 LIBS:device
@@
 SPI ADC 8 Channel
 $Comp
-L MCP3008 U5
-U 1 1 563769CE
-P 4800 2650
-F 0 "U5" H 4850 3000 60  0000 C CNN
-F 1 "MCP3008" H 4900 1900 60  0000 C CNN
-F 2 "REInnovationFootprint:DIP-16__300_ELL_lg_pad" H 5000 2650 60  0001 C CNN
-F 3 "" H 5000 2650 60  0000 C CNN
-	1    4800 2650
-	1    0    0    -1
-$EndComp
-$Comp
 L CONN_02X08 P13
 U 1 1 563769D5
@@
 P 6050 2200
 F 0 "C8" H 6100 2300 50  0000 L CNN
-F 1 "1000n" H 6100 2100 50  0000 L CNN
+F 1 "1u" H 6100 2100 50  0000 L CNN
 F 2 "matts_components:C1_wide_lg_pad_2" H 6050 2200 60  0001 C CNN
 F 3 "" H 6050 2200 60  0000 C CNN
@@
 $EndComp
 $Comp
-L MCP3008 U6
-U 1 1 56376A0A
-P 4800 3900
-F 0 "U6" H 4850 4250 60  0000 C CNN
-F 1 "MCP3008" H 4900 3200 60  0000 C CNN
-F 2 "REInnovationFootprint:DIP-16__300_ELL_lg_pad" H 5000 3900 60  0001 C CNN
-F 3 "" H 5000 3900 60  0000 C CNN
-	1    4800 3900
-	1    0    0    -1
-$EndComp
-$Comp
 L CONN_02X08 P14
 U 1 1 56376A11
@@
 P 6000 3400
 F 0 "C7" H 6050 3500 50  0000 L CNN
-F 1 "1000n" H 6050 3300 50  0000 L CNN
+F 1 "1u" H 6050 3300 50  0000 L CNN
 F 2 "matts_components:C1_wide_lg_pad_2" H 6000 3400 60  0001 C CNN
 F 3 "" H 6000 3400 60  0000 C CNN
@@
 P 7650 5500
 F 0 "U7" H 7650 5800 60  0000 C CNN
-F 1 "MCP4802" H 7600 5150 60  0000 C CNN
+F 1 "MCP4812" H 7600 5150 60  0000 C CNN
 F 2 "REInnovationFootprint:DIP-8_300_ELL" H 7650 5500 60  0001 C CNN
 F 3 "http://ww1.microchip.com/downloads/en/DeviceDoc/22249A.pdf" H 7650 5500 60  0001 C CNN
@@
 F 3 "" H 7750 3050 60  0000 C CNN
 	1    7750 3050
-	1    0    0    -1
+	1    0    0    1
 $EndComp
 Wire Wire Line
@@
 	5650 3450 5650 3950
 Wire Wire Line
-	5650 3950 5350 3950
+	5350 3950 5750 3950
 Wire Wire Line
 	3700 4350 3500 4350
@@
 Wire Wire Line
 	5350 3000 7550 3000
-Wire Wire Line
-	5350 3100 7550 3100
 Wire Wire Line
 	6850 3200 7550 3200
@@
 Connection ~ 6750 3000
 Wire Wire Line
-	7300 5500 7200 5500
-Wire Wire Line
-	7200 5500 7200 3300
-Wire Wire Line
-	7200 3300 7550 3300
+	7100 5500 7300 5500
 Wire Wire Line
 	6550 5600 7300 5600
@@
 P 7900 4850
 F 0 "C9" H 7950 4950 50  0000 L CNN
-F 1 "100n" H 7950 4750 50  0000 L CNN
+F 1 "1u" H 7950 4750 50  0000 L CNN
 F 2 "matts_components:C1_wide_lg_pad_2" H 7900 4850 60  0001 C CNN
 F 3 "" H 7900 4850 60  0000 C CNN
@@
 Text HLabel 9850 5750 3    60   Input ~ 0
 GND
+$Comp
+L MCP3008_16pin U6
+U 1 1 599191BF
+P 5150 4050
+F 0 "U6" H 4700 4500 50  0000 C CNN
+F 1 "MCP3008" H 4950 3500 50  0000 C CNN
+F 2 "REInnovationFootprint:DIP-16__300_ELL_lg_pad" H 5050 3950 50  0001 C CNN
+F 3 "" H 5150 4050 50  0000 C CNN
+	1    5150 4050
+	1    0    0    -1
+$EndComp
+$Comp
+L MCP3008_16pin U5
+U 1 1 5991993D
+P 5150 2800
+F 0 "U5" H 4700 3250 50  0000 C CNN
+F 1 "MCP3008" H 4950 2250 50  0000 C CNN
+F 2 "REInnovationFootprint:DIP-16__300_ELL_lg_pad" H 5050 2700 50  0001 C CNN
+F 3 "" H 5150 2800 50  0000 C CNN
+	1    5150 2800
+	1    0    0    -1
+$EndComp
+Text HLabel 5750 3950 2    60   Input ~ 0
+GND
+Connection ~ 5650 3950
+Text HLabel 5500 2100 2    60   Input ~ 0
+GND
+Wire Wire Line
+	5500 2100 5350 2100
+Wire Wire Line
+	5350 2100 5350 2200
+Connection ~ 5350 2200
+$Comp
+L R R55
+U 1 1 5991CDDF
+P 7350 2250
+F 0 "R55" V 7430 2250 50  0000 C CNN
+F 1 "100k" V 7350 2250 50  0000 C CNN
+F 2 "REInnovationFootprint:TH_Resistor_1" V 7280 2250 50  0001 C CNN
+F 3 "" H 7350 2250 50  0000 C CNN
+	1    7350 2250
+	1    0    0    -1
+$EndComp
+$Comp
+L R R56
+U 1 1 5991CF0E
+P 7550 2250
+F 0 "R56" V 7630 2250 50  0000 C CNN
+F 1 "100k" V 7550 2250 50  0000 C CNN
+F 2 "REInnovationFootprint:TH_Resistor_1" V 7480 2250 50  0001 C CNN
+F 3 "" H 7550 2250 50  0000 C CNN
+	1    7550 2250
+	1    0    0    -1
+$EndComp
+Wire Wire Line
+	7350 2400 7350 3300
+Wire Wire Line
+	7450 2500 7450 3200
+Connection ~ 7450 3200
+Text HLabel 7300 1950 0    60   Input ~ 0
++3V3
+Wire Wire Line
+	7300 1950 8050 1950
+Wire Wire Line
+	7550 1950 7550 2100
+Wire Wire Line
+	7350 2100 7350 1950
+Connection ~ 7350 1950
+Text Notes 8250 1950 0    60   ~ 0
+~CS~ PULL UP
+Wire Wire Line
+	7350 3300 7550 3300
+Wire Wire Line
+	5350 3100 7350 3100
+Connection ~ 7350 3100
+Wire Wire Line
+	7450 2500 7550 2500
+Wire Wire Line
+	7550 2500 7550 2400
+Wire Wire Line
+	7550 3100 7500 3100
+Wire Wire Line
+	7500 3100 7500 4550
+Wire Wire Line
+	7500 4550 7100 4550
+Wire Wire Line
+	7100 4550 7100 5500
+$Comp
+L R R57
+U 1 1 59921707
+P 8050 2250
+F 0 "R57" V 8130 2250 50  0000 C CNN
+F 1 "100k" V 8050 2250 50  0000 C CNN
+F 2 "REInnovationFootprint:TH_Resistor_1" V 7980 2250 50  0001 C CNN
+F 3 "" H 8050 2250 50  0000 C CNN
+	1    8050 2250
+	1    0    0    -1
+$EndComp
+Wire Wire Line
+	8050 2400 8050 3700
+Wire Wire Line
+	8050 3700 7500 3700
+Connection ~ 7500 3700
+Wire Wire Line
+	8050 1950 8050 2100
+Connection ~ 7550 1950
 $EndSCHEMATC
