File: Hardware/PCB Design/KiCAD Files/IO.sch (KiCad schematic (older format))
At the start: 16 parts, among them P18 DIO_OUTPUT, P19 PULL_UP, P20 PULL_DOWN, P21 DIO_INPUT

Commit message: Version 3 revision
Added 3A switching 5V supply and Capacitors axial and radial
Parts:
- P18, P19, P20: footprint Pin_Headers:Pin_Header_Straight_2x12 -> REInnovationFootprint:Pin_Header_Straight_2x12
Changed lines of the file:
@@
 LIBS:contrib
 LIBS:valves
+LIBS:oBeMs_Pulse_PCB-cache
 LIBS:matts_components
-LIBS:oBeMs_Pulse_PCB-cache
 EELAYER 25 0
 EELAYER END
@@
 Title "oBeMs Open Pulse Monitor Unit"
 Date "2015-11-01"
-Rev "2"
+Rev "3"
 Comp "T4 Sustainability"
 Comment1 "PCB design by RE-Innovation"
@@
 $EndComp
 $Comp
-L +3.3V-RESCUE-oBeMs_Pulse_PCB #PWR027
+L +3.3V-RESCUE-oBeMs_Pulse_PCB #PWR029
 U 1 1 563790C9
 P 5050 900
-AR Path="/56378529/563790C9" Ref="#PWR027"  Part="1"
-AR Path="/5637E9E0/563790C9" Ref="#PWR029"  Part="1"
-AR Path="/5637EAA2/563790C9" Ref="#PWR031"  Part="1"
+AR Path="/56378529/563790C9" Ref="#PWR029"  Part="1"
+AR Path="/5637E9E0/563790C9" Ref="#PWR031"  Part="1"
+AR Path="/5637EAA2/563790C9" Ref="#PWR033"  Part="1"
 AR Path="/5637EAA4/563790C9" Ref="#PWR041"  Part="1"
-F 0 "#PWR031" H 5050 860 30  0001 C CNN
+F 0 "#PWR033" H 5050 860 30  0001 C CNN
 F 1 "+3.3V" H 5050 1010 30  0000 C CNN
 F 2 "" H 5050 900 60  0000 C CNN
@@
 DIO
 $Comp
-L GND-RESCUE-oBeMs_Pulse_PCB #PWR028
+L GND-RESCUE-oBeMs_Pulse_PCB #PWR030
 U 1 1 563790D7
 P 5200 4600
-AR Path="/56378529/563790D7" Ref="#PWR028"  Part="1"
-AR Path="/5637E9E0/563790D7" Ref="#PWR030"  Part="1"
-AR Path="/5637EAA2/563790D7" Ref="#PWR032"  Part="1"
+AR Path="/56378529/563790D7" Ref="#PWR030"  Part="1"
+AR Path="/5637E9E0/563790D7" Ref="#PWR032"  Part="1"
+AR Path="/5637EAA2/563790D7" Ref="#PWR034"  Part="1"
 AR Path="/5637EAA4/563790D7" Ref="#PWR042"  Part="1"
-F 0 "#PWR032" H 5200 4600 30  0001 C CNN
+F 0 "#PWR034" H 5200 4600 30  0001 C CNN
 F 1 "GND" H 5200 4530 30  0001 C CNN
 F 2 "" H 5200 4600 60  0000 C CNN
@@
 F 0 "P27" H 5200 2600 50  0000 C CNN
 F 1 "PULL_UP" V 5200 1950 50  0000 C CNN
-F 2 "Pin_Headers:Pin_Header_Straight_2x12" H 5200 750 60  0001 C CNN
+F 2 "REInnovationFootprint:Pin_Header_Straight_2x12" H 5200 750 60  0001 C CNN
 F 3 "" H 5200 750 60  0000 C CNN
 F 4 "~" H 5200 1950 60  0001 C CNN "Description"
@@
 F 0 "P28" H 5200 4650 50  0000 C CNN
 F 1 "PULL_DOWN" V 5200 4000 50  0000 C CNN
-F 2 "Pin_Headers:Pin_Header_Straight_2x12" H 5200 2800 60  0001 C CNN
+F 2 "REInnovationFootprint:Pin_Header_Straight_2x12" H 5200 2800 60  0001 C CNN
 F 3 "" H 5200 2800 60  0000 C CNN
 F 4 "~" H 5200 4000 60  0001 C CNN "Description"
@@
 F 0 "P26" H 3750 3600 50  0000 C CNN
 F 1 "DIO_OUTPUT" V 4100 2950 50  0000 C CNN
-F 2 "Pin_Headers:Pin_Header_Straight_2x12" H 3750 1750 60  0001 C CNN
+F 2 "REInnovationFootprint:Pin_Header_Straight_2x12" H 3750 1750 60  0001 C CNN
 F 3 "" H 3750 1750 60  0000 C CNN
 F 4 "~" H 3750 2950 60  0001 C CNN "Description"

Commit message: Updates from email 21/12/15
Parts:
- P20: value PULL_DOWN -> GROUND
Changed lines of the file:
@@
 LIBS:contrib
 LIBS:valves
+LIBS:matts_components
 LIBS:oBeMs_Pulse_PCB-cache
-LIBS:matts_components
 EELAYER 25 0
 EELAYER END
@@
 Sheet 9 10
 Title "oBeMs Open Pulse Monitor Unit"
-Date "2015-11-01"
-Rev "3"
+Date "2015-12-21"
+Rev "4"
 Comp "T4 Sustainability"
 Comment1 "PCB design by RE-Innovation"
@@
 $EndComp
 $Comp
-L +3.3V-RESCUE-oBeMs_Pulse_PCB #PWR029
+L +3.3V-RESCUE-oBeMs_Pulse_PCB #PWR030
 U 1 1 563790C9
 P 5050 900
-AR Path="/56378529/563790C9" Ref="#PWR029"  Part="1"
-AR Path="/5637E9E0/563790C9" Ref="#PWR031"  Part="1"
-AR Path="/5637EAA2/563790C9" Ref="#PWR033"  Part="1"
+AR Path="/56378529/563790C9" Ref="#PWR030"  Part="1"
+AR Path="/5637E9E0/563790C9" Ref="#PWR032"  Part="1"
+AR Path="/5637EAA2/563790C9" Ref="#PWR034"  Part="1"
 AR Path="/5637EAA4/563790C9" Ref="#PWR041"  Part="1"
-F 0 "#PWR033" H 5050 860 30  0001 C CNN
+F 0 "#PWR034" H 5050 860 30  0001 C CNN
 F 1 "+3.3V" H 5050 1010 30  0000 C CNN
 F 2 "" H 5050 900 60  0000 C CNN
@@
 DIO
 $Comp
-L GND-RESCUE-oBeMs_Pulse_PCB #PWR030
+L GND-RESCUE-oBeMs_Pulse_PCB #PWR031
 U 1 1 563790D7
 P 5200 4600
-AR Path="/56378529/563790D7" Ref="#PWR030"  Part="1"
-AR Path="/5637E9E0/563790D7" Ref="#PWR032"  Part="1"
-AR Path="/5637EAA2/563790D7" Ref="#PWR034"  Part="1"
+AR Path="/56378529/563790D7" Ref="#PWR031"  Part="1"
+AR Path="/5637E9E0/563790D7" Ref="#PWR033"  Part="1"
+AR Path="/5637EAA2/563790D7" Ref="#PWR035"  Part="1"
 AR Path="/5637EAA4/563790D7" Ref="#PWR042"  Part="1"
-F 0 "#PWR034" H 5200 4600 30  0001 C CNN
+F 0 "#PWR035" H 5200 4600 30  0001 C CNN
 F 1 "GND" H 5200 4530 30  0001 C CNN
 F 2 "" H 5200 4600 60  0000 C CNN
@@
 AR Path="/5637EAA4/56379AE8" Ref="P32"  Part="1"
 F 0 "P28" H 5200 4650 50  0000 C CNN
-F 1 "PULL_DOWN" V 5200 4000 50  0000 C CNN
+F 1 "GROUND" V 5200 4000 50  0000 C CNN
 F 2 "REInnovationFootprint:Pin_Header_Straight_2x12" H 5200 2800 60  0001 C CNN
 F 3 "" H 5200 2800 60  0000 C CNN

Commit message: Rev 6. Final changes before PCB v0000 done
Connections:
- net +3.3V renamed +3V3
Changed lines of the file:
@@
 encoding utf-8
 Sheet 9 10
-Title "oBeMs Open Pulse Monitor Unit"
-Date "2015-12-22"
-Rev "5"
+Title "oBeMS Open Interface Board 0001"
+Date "2015-12-23"
+Rev "6"
 Comp "T4 Sustainability"
-Comment1 "PCB design by RE-Innovation"
+Comment1 "PCB design by T4 Sustainability/RE-Innovation"
 Comment2 ""
 Comment3 ""
@@
 	1    0    0    -1
 $EndComp
-$Comp
-L +3.3V-RESCUE-oBeMs_Pulse_PCB #PWR030
-U 1 1 563790C9
-P 5050 900
-AR Path="/56378529/563790C9" Ref="#PWR030"  Part="1"
-AR Path="/5637E9E0/563790C9" Ref="#PWR032"  Part="1"
-AR Path="/5637EAA2/563790C9" Ref="#PWR034"  Part="1"
-AR Path="/5637EAA4/563790C9" Ref="#PWR041"  Part="1"
-F 0 "#PWR034" H 5050 860 30  0001 C CNN
-F 1 "+3.3V" H 5050 1010 30  0000 C CNN
-F 2 "" H 5050 900 60  0000 C CNN
-F 3 "" H 5050 900 60  0000 C CNN
-	1    5050 900
-	1    0    0    -1
-$EndComp
 Text Notes 4000 2000 0    60   ~ 0
 DIO
-$Comp
-L GND-RESCUE-oBeMs_Pulse_PCB #PWR031
-U 1 1 563790D7
-P 5200 4600
-AR Path="/56378529/563790D7" Ref="#PWR031"  Part="1"
-AR Path="/5637E9E0/563790D7" Ref="#PWR033"  Part="1"
-AR Path="/5637EAA2/563790D7" Ref="#PWR035"  Part="1"
-AR Path="/5637EAA4/563790D7" Ref="#PWR042"  Part="1"
-F 0 "#PWR035" H 5200 4600 30  0001 C CNN
-F 1 "GND" H 5200 4530 30  0001 C CNN
-F 2 "" H 5200 4600 60  0000 C CNN
-F 3 "" H 5200 4600 60  0000 C CNN
-	1    5200 4600
-	-1   0    0    -1
-$EndComp
 $Comp
 L CONN_02X12 P19
@@
 Connection ~ 4500 950
 Wire Wire Line
-	5050 900  5050 950
+	5050 750  5050 950
 Connection ~ 5050 950
+Text HLabel 4900 750  0    60   Input ~ 0
++3V3
+Text HLabel 5200 4600 3    60   Input ~ 0
+GND
+Wire Wire Line
+	4900 750  5050 750
 $EndSCHEMATC

Commit message: Changes for v0001
Multiple PCb changes. 50Pcs ordered
Parts:
- P19, P20: footprint REInnovationFootprint:Pin_Header_Straight_2x12 -> REInnovationFootprint:Pin_Header_Straight_2x12_SM_Connect
Changed lines of the file:
@@
 EESchema Schematic File Version 2
-LIBS:oBeMs_Pulse_PCB-rescue
 LIBS:power
 LIBS:device
@@
 $Descr A4 11693 8268
 encoding utf-8
-Sheet 9 10
+Sheet 8 10
 Title "oBeMS Open Interface Board 0001"
 Date "2015-12-23"
@@
 F 0 "P27" H 5200 2600 50  0000 C CNN
 F 1 "PULL_UP" V 5200 1950 50  0000 C CNN
-F 2 "REInnovationFootprint:Pin_Header_Straight_2x12" H 5200 750 60  0001 C CNN
+F 2 "REInnovationFootprint:Pin_Header_Straight_2x12_SM_Connect" H 5200 750 60  0001 C CNN
 F 3 "" H 5200 750 60  0000 C CNN
 F 4 "~" H 5200 1950 60  0001 C CNN "Description"
@@
 F 0 "P28" H 5200 4650 50  0000 C CNN
 F 1 "GROUND" V 5200 4000 50  0000 C CNN
-F 2 "REInnovationFootprint:Pin_Header_Straight_2x12" H 5200 2800 60  0001 C CNN
+F 2 "REInnovationFootprint:Pin_Header_Straight_2x12_SM_Connect" H 5200 2800 60  0001 C CNN
 F 3 "" H 5200 2800 60  0000 C CNN
 F 4 "~" H 5200 4000 60  0001 C CNN "Description"
