File: Hardware/PCB Design/KiCAD Files/LED.sch (KiCad schematic (older format))
At the start: 16 parts

Commit message: Rev 6. Final changes before PCB v0000 done
Changed lines of the file:
@@
 encoding utf-8
 Sheet 5 10
-Title "oBeMs Open Pulse Monitor Unit"
-Date "2015-12-22"
-Rev "5"
+Title "oBeMS Open Interface Board 0001"
+Date "2015-12-23"
+Rev "6"
 Comp "T4 Sustainability"
-Comment1 "PCB design by RE-Innovation"
+Comment1 "PCB design by T4 Sustainability/RE-Innovation"
 Comment2 ""
 Comment3 ""
@@
 	1    4400 3900
 	0    1    1    0
-$EndComp
-$Comp
-L GND-RESCUE-oBeMs_Pulse_PCB #PWR017
-U 1 1 56370E51
-P 4250 4250
-F 0 "#PWR017" H 4250 4250 30  0001 C CNN
-F 1 "GND" H 4250 4180 30  0001 C CNN
-F 2 "" H 4250 4250 60  0000 C CNN
-F 3 "" H 4250 4250 60  0000 C CNN
-	1    4250 4250
-	1    0    0    -1
 $EndComp
 $Comp
@@
 Wire Wire Line
 	4700 2650 4700 2850
+Text HLabel 4250 4250 0    60   Input ~ 0
+GND
 $EndSCHEMATC
