File: Hardware/PCB Design/KiCAD Files/PrototypeArea.sch (KiCad schematic (older format))
At the start: 1 part, among them P36 PROTOTYPING_AREA

Commit message: Updates from email 21/12/15
Connections:
- net GND: no longer names the net of P36.2 (P2)
- no-connect marks 15 -> 16
Changed lines of the file:
@@
 LIBS:contrib
 LIBS:valves
+LIBS:matts_components
 LIBS:oBeMs_Pulse_PCB-cache
-LIBS:matts_components
 EELAYER 25 0
 EELAYER END
@@
 encoding utf-8
 Sheet 10 10
-Title ""
-Date ""
-Rev "3"
-Comp ""
-Comment1 ""
+Title "oBeMs Open Pulse Monitor Unit"
+Date "2015-12-21"
+Rev "4"
+Comp "T4 Sustainability"
+Comment1 "PCB design by RE-Innovation"
 Comment2 ""
 Comment3 ""
@@
 NoConn ~ 4850 3300
 NoConn ~ 4850 3200
-$Comp
-L GND-RESCUE-oBeMs_Pulse_PCB #PWR043
-U 1 1 56388993
-P 4700 3150
-AR Path="/56388993" Ref="#PWR043"  Part="1"
-AR Path="/56384A5B/56388993" Ref="#PWR035"  Part="1"
-F 0 "#PWR035" H 4700 2900 50  0001 C CNN
-F 1 "GND" H 4700 3000 50  0000 C CNN
-F 2 "" H 4700 3150 60  0000 C CNN
-F 3 "" H 4700 3150 60  0000 C CNN
-	1    4700 3150
-	1    0    0    -1
-$EndComp
-Wire Wire Line
-	4850 3100 4700 3100
-Wire Wire Line
-	4700 3100 4700 3150
 NoConn ~ 4850 3000
+NoConn ~ 4850 3100
 $EndSCHEMATC

Commit message: More small changes 22/12/15
Parts:
- added P9: V?, matts_components:SIL-3_solder_connect, symbol CONN_01X03
- P36: footprint REInnovationFootprint:PROTO_AREA -> REInnovationFootprint:PROTO_AREA_16x14
Connections:
- net at P36.1 (P1): now also P9.2 (P2)
- net GND: now reaches P36.2 (P2)
- new net +3.3V: P9.1 (P1)
- new net +5V: P9.3 (P3)
- no-connect marks 16 -> 14
Changed lines of the file:
@@
 LIBS:contrib
 LIBS:valves
+LIBS:oBeMs_Pulse_PCB-cache
 LIBS:matts_components
-LIBS:oBeMs_Pulse_PCB-cache
 EELAYER 25 0
 EELAYER END
@@
 Sheet 10 10
 Title "oBeMs Open Pulse Monitor Unit"
-Date "2015-12-21"
-Rev "4"
+Date "2015-12-22"
+Rev "5"
 Comp "T4 Sustainability"
 Comment1 "PCB design by RE-Innovation"
@@
 F 0 "P36" H 5050 4600 50  0000 C CNN
 F 1 "PROTOTYPING_AREA" V 5150 3750 50  0000 C CNN
-F 2 "REInnovationFootprint:PROTO_AREA" H 5050 3750 60  0001 C CNN
+F 2 "REInnovationFootprint:PROTO_AREA_16x14" H 5050 3750 60  0001 C CNN
 F 3 "" H 5050 3750 60  0000 C CNN
 	1    5050 3750
@@
 NoConn ~ 4850 3300
 NoConn ~ 4850 3200
-NoConn ~ 4850 3000
-NoConn ~ 4850 3100
+$Comp
+L GND #PWR036
+U 1 1 5679222E
+P 4300 3300
+F 0 "#PWR036" H 4300 3050 50  0001 C CNN
+F 1 "GND" H 4300 3150 50  0000 C CNN
+F 2 "" H 4300 3300 50  0000 C CNN
+F 3 "" H 4300 3300 50  0000 C CNN
+	1    4300 3300
+	1    0    0    -1
+$EndComp
+$Comp
+L +5V #PWR037
+U 1 1 5679225A
+P 4350 2850
+F 0 "#PWR037" H 4350 2700 50  0001 C CNN
+F 1 "+5V" H 4350 2990 50  0000 C CNN
+F 2 "" H 4350 2850 50  0000 C CNN
+F 3 "" H 4350 2850 50  0000 C CNN
+	1    4350 2850
+	1    0    0    -1
+$EndComp
+$Comp
+L CONN_01X03 P9
+U 1 1 56792277
+P 4050 2700
+F 0 "P9" H 4050 2900 50  0000 C CNN
+F 1 "V?" V 4150 2700 50  0000 C CNN
+F 2 "matts_components:SIL-3_solder_connect" H 4050 2700 50  0001 C CNN
+F 3 "" H 4050 2700 50  0000 C CNN
+	1    4050 2700
+	0    -1   -1   0
+$EndComp
+Wire Wire Line
+	4850 3100 4300 3100
+Wire Wire Line
+	4300 3100 4300 3300
+Wire Wire Line
+	4850 3000 4050 3000
+Wire Wire Line
+	4050 3000 4050 2900
+Wire Wire Line
+	4150 2900 4350 2900
+Wire Wire Line
+	4350 2900 4350 2850
+Wire Wire Line
+	3700 2900 3950 2900
+Wire Wire Line
+	3700 2800 3700 2900
+$Comp
+L +3.3V-RESCUE-oBeMs_Pulse_PCB #PWR038
+U 1 1 56794A4F
+P 3700 2800
+F 0 "#PWR038" H 3700 2760 30  0001 C CNN
+F 1 "+3.3V" H 3700 2910 30  0000 C CNN
+F 2 "" H 3700 2800 60  0000 C CNN
+F 3 "" H 3700 2800 60  0000 C CNN
+	1    3700 2800
+	1    0    0    -1
+$EndComp
 $EndSCHEMATC

Commit message: Rev 6. Final changes before PCB v0000 done
Parts:
- removed P36: PROTOTYPING_AREA, REInnovationFootprint:PROTO_AREA_16x14, symbol CONN_01X16
- added P31: V2?, REInnovationFootprint:SIL-3_solder_connect, symbol CONN_01X03
- added P36: PROTOTYPING_AREA, REInnovationFootprint:PROTO_AREA_16x14, symbol CONN_01X18
- P9: value V? -> V1?; footprint matts_components:SIL-3_solder_connect -> REInnovationFootprint:SIL-3_solder_connect
Connections:
- net GND: now also P36.18 (P18), P36.2 (P2)
- net at P9.2 (P2): now also P36.1 (P1)
- net +3.3V renamed +3V3
- net +3V3: now also P31.1 (P1)
- net +5V renamed 5V
- net 5V: now also P31.3 (P3)
- new net: P31.2 (P2), P36.17 (P17)
Changed lines of the file:
@@
 encoding utf-8
 Sheet 10 10
-Title "oBeMs Open Pulse Monitor Unit"
-Date "2015-12-22"
-Rev "5"
+Title "oBeMS Open Interface Board 0001"
+Date "2015-12-23"
+Rev "6"
 Comp "T4 Sustainability"
-Comment1 "PCB design by RE-Innovation"
+Comment1 "PCB design by T4 Sustainability/RE-Innovation"
 Comment2 ""
 Comment3 ""
 Comment4 ""
 $EndDescr
-$Comp
-L CONN_01X16 P36
-U 1 1 5638891D
-P 5050 3750
-F 0 "P36" H 5050 4600 50  0000 C CNN
-F 1 "PROTOTYPING_AREA" V 5150 3750 50  0000 C CNN
-F 2 "REInnovationFootprint:PROTO_AREA_16x14" H 5050 3750 60  0001 C CNN
-F 3 "" H 5050 3750 60  0000 C CNN
-	1    5050 3750
-	1    0    0    -1
-$EndComp
 NoConn ~ 4850 4500
 NoConn ~ 4850 4400
@@
 NoConn ~ 4850 3200
 $Comp
-L GND #PWR036
-U 1 1 5679222E
-P 4300 3300
-F 0 "#PWR036" H 4300 3050 50  0001 C CNN
-F 1 "GND" H 4300 3150 50  0000 C CNN
-F 2 "" H 4300 3300 50  0000 C CNN
-F 3 "" H 4300 3300 50  0000 C CNN
-	1    4300 3300
-	1    0    0    -1
-$EndComp
-$Comp
-L +5V #PWR037
-U 1 1 5679225A
-P 4350 2850
-F 0 "#PWR037" H 4350 2700 50  0001 C CNN
-F 1 "+5V" H 4350 2990 50  0000 C CNN
-F 2 "" H 4350 2850 50  0000 C CNN
-F 3 "" H 4350 2850 50  0000 C CNN
-	1    4350 2850
-	1    0    0    -1
-$EndComp
-$Comp
 L CONN_01X03 P9
 U 1 1 56792277
 P 4050 2700
 F 0 "P9" H 4050 2900 50  0000 C CNN
-F 1 "V?" V 4150 2700 50  0000 C CNN
-F 2 "matts_components:SIL-3_solder_connect" H 4050 2700 50  0001 C CNN
+F 1 "V1?" V 4150 2700 50  0000 C CNN
+F 2 "REInnovationFootprint:SIL-3_solder_connect" H 4050 2700 50  0001 C CNN
 F 3 "" H 4050 2700 50  0000 C CNN
 	1    4050 2700
@@
 $EndComp
 Wire Wire Line
-	4850 3100 4300 3100
-Wire Wire Line
-	4300 3100 4300 3300
+	4250 3100 4850 3100
 Wire Wire Line
 	4850 3000 4050 3000
@@
 Wire Wire Line
 	3700 2800 3700 2900
+Text HLabel 3700 2800 0    60   Input ~ 0
++3V3
+Text HLabel 4350 2850 2    60   Input ~ 0
+5V
+Text HLabel 4250 3100 0    60   Input ~ 0
+GND
 $Comp
-L +3.3V-RESCUE-oBeMs_Pulse_PCB #PWR038
-U 1 1 56794A4F
-P 3700 2800
-F 0 "#PWR038" H 3700 2760 30  0001 C CNN
-F 1 "+3.3V" H 3700 2910 30  0000 C CNN
-F 2 "" H 3700 2800 60  0000 C CNN
-F 3 "" H 3700 2800 60  0000 C CNN
-	1    3700 2800
+L CONN_01X18 P36
+U 1 1 567AD735
+P 5050 3850
+F 0 "P36" H 5050 4800 50  0000 C CNN
+F 1 "PROTOTYPING_AREA" V 5150 3850 50  0000 C CNN
+F 2 "REInnovationFootprint:PROTO_AREA_16x14" H 5050 3850 50  0001 C CNN
+F 3 "" H 5050 3850 50  0000 C CNN
+	1    5050 3850
 	1    0    0    -1
 $EndComp
+$Comp
+L CONN_01X03 P31
+U 1 1 567AD838
+P 4050 4300
+F 0 "P31" H 4050 4500 50  0000 C CNN
+F 1 "V2?" V 4150 4300 50  0000 C CNN
+F 2 "REInnovationFootprint:SIL-3_solder_connect" H 4050 4300 50  0001 C CNN
+F 3 "" H 4050 4300 50  0000 C CNN
+	1    4050 4300
+	0    -1   -1   0
+$EndComp
+Wire Wire Line
+	4250 4700 4850 4700
+Wire Wire Line
+	4850 4600 4050 4600
+Wire Wire Line
+	4050 4600 4050 4500
+Wire Wire Line
+	4150 4500 4350 4500
+Wire Wire Line
+	4350 4500 4350 4450
+Wire Wire Line
+	3700 4500 3950 4500
+Wire Wire Line
+	3700 4400 3700 4500
+Text HLabel 3700 4400 0    60   Input ~ 0
++3V3
+Text HLabel 4350 4450 2    60   Input ~ 0
+5V
+Text HLabel 4250 4700 0    60   Input ~ 0
+GND
 $EndSCHEMATC
