File: Hardware/PCB Design/KiCAD Files/WDT.sch (KiCad schematic (older format))
At the start: 25 parts, among them Q1 BC546, Q2 BC556, U3 TLC555, U4 4017

Commit message: Version 3 revision
Added 3A switching 5V supply and Capacitors axial and radial
Parts:
- C6: footprint matts_components:C2V8_large_pads -> REInnovationFootprint:C2V8_VandA
Changed lines of the file:
@@
 LIBS:contrib
 LIBS:valves
+LIBS:oBeMs_Pulse_PCB-cache
 LIBS:matts_components
-LIBS:oBeMs_Pulse_PCB-cache
 EELAYER 25 0
 EELAYER END
@@
 Title "oBeMs Open Pulse Monitor Unit"
 Date "2015-11-01"
-Rev "2"
+Rev "3"
 Comp "T4 Sustainability"
 Comment1 "PCB design by RE-Innovation"
@@
 F 0 "C6" H 6150 3000 50  0000 L CNN
 F 1 "47u" H 6150 2800 50  0000 L CNN
-F 2 "matts_components:C2V8_large_pads" H 6100 2900 60  0001 C CNN
+F 2 "REInnovationFootprint:C2V8_VandA" H 6100 2900 60  0001 C CNN
 F 3 "" H 6100 2900 60  0000 C CNN
 	1    6100 2900

Commit message: Updates from email 21/12/15
Parts:
- removed R10, R55, R56: 120, REInnovationFootprint:TH_Resistor_1, symbol R-RESCUE-oBeMs_Pulse_PCB
- R6: value 120 -> 100
Connections:
- net VDD: now also Q2.3 (E); no longer Q2.1 (C)
- net at C3.1, R2.1: now also Q2.1 (C); no longer Q2.3 (E)
- net at U4.3 (Q0): now also D12.1 (A)
- net at U4.6 (Q7): now also D13.1 (A)
- net at U4.9 (Q8): now also D14.1 (A)
Changed lines of the file:
@@
 LIBS:contrib
 LIBS:valves
+LIBS:matts_components
 LIBS:oBeMs_Pulse_PCB-cache
-LIBS:matts_components
 EELAYER 25 0
 EELAYER END
@@
 Sheet 4 10
 Title "oBeMs Open Pulse Monitor Unit"
-Date "2015-11-01"
-Rev "3"
+Date "2015-12-21"
+Rev "4"
 Comp "T4 Sustainability"
 Comment1 "PCB design by RE-Innovation"
@@
 P 7600 3800
 F 0 "R6" V 7680 3800 50  0000 C CNN
-F 1 "120" V 7600 3800 50  0000 C CNN
+F 1 "100" V 7600 3800 50  0000 C CNN
 F 2 "REInnovationFootprint:TH_Resistor_1" H 7600 3800 60  0001 C CNN
 F 3 "" H 7600 3800 60  0000 C CNN
@@
 +3.3V
 $Comp
-L R-RESCUE-oBeMs_Pulse_PCB R10
-U 1 1 563A562D
-P 6600 3600
-F 0 "R10" V 6680 3600 50  0000 C CNN
-F 1 "120" V 6600 3600 50  0000 C CNN
-F 2 "REInnovationFootprint:TH_Resistor_1" H 6600 3600 60  0001 C CNN
-F 3 "" H 6600 3600 60  0000 C CNN
-F 4 "Value" H 6600 3600 60  0001 C CNN "Description"
-F 5 "Value" H 6600 3600 60  0001 C CNN "Notes"
-F 6 "Value" H 6600 3600 60  0001 C CNN "Manufacturer"
-F 7 "Value" H 6600 3600 60  0001 C CNN "Manufacturer Part No"
-F 8 "Value" H 6600 3600 60  0001 C CNN "Supplier 1"
-F 9 "Value" H 6600 3600 60  0001 C CNN "Supplier 1 Part No"
-F 10 "Value" H 6600 3600 60  0001 C CNN "Supplier 2"
-F 11 "Value" H 6600 3600 60  0001 C CNN "Supplier 2 Part No"
-	1    6600 3600
-	1    0    0    1
-$EndComp
-$Comp
 L LED-RESCUE-oBeMs_Pulse_PCB D12
 U 1 1 563A5633
@@
 $EndComp
 Wire Wire Line
-	6600 3250 6600 3350
-Wire Wire Line
-	6600 3850 6600 4000
+	6600 3250 6600 4000
 Wire Wire Line
 	4850 4100 5150 4100
@@
 P 3800 3950
 F 0 "Q2" H 3800 3800 60  0000 R CNN
-F 1 "BC556" H 3800 4100 60  0000 R CNN
+F 1 "BC556" H 4300 3850 60  0000 R CNN
 F 2 "matts_components:TO92-PNP_large_pad" H 3800 3950 60  0001 C CNN
 F 3 "" H 3800 3950 60  0000 C CNN
 	1    3800 3950
-	1    0    0    -1
+	1    0    0    1
 $EndComp
 Wire Wire Line
@@
 	7600 4600 7750 4600
 Connection ~ 7600 4600
-$Comp
-L R-RESCUE-oBeMs_Pulse_PCB R55
-U 1 1 563A651A
-P 6900 3600
-F 0 "R55" V 6980 3600 50  0000 C CNN
-F 1 "120" V 6900 3600 50  0000 C CNN
-F 2 "REInnovationFootprint:TH_Resistor_1" H 6900 3600 60  0001 C CNN
-F 3 "" H 6900 3600 60  0000 C CNN
-F 4 "Value" H 6900 3600 60  0001 C CNN "Description"
-F 5 "Value" H 6900 3600 60  0001 C CNN "Notes"
-F 6 "Value" H 6900 3600 60  0001 C CNN "Manufacturer"
-F 7 "Value" H 6900 3600 60  0001 C CNN "Manufacturer Part No"
-F 8 "Value" H 6900 3600 60  0001 C CNN "Supplier 1"
-F 9 "Value" H 6900 3600 60  0001 C CNN "Supplier 1 Part No"
-F 10 "Value" H 6900 3600 60  0001 C CNN "Supplier 2"
-F 11 "Value" H 6900 3600 60  0001 C CNN "Supplier 2 Part No"
-	1    6900 3600
-	1    0    0    1
-$EndComp
 $Comp
 L LED-RESCUE-oBeMs_Pulse_PCB D13
@@
 $EndComp
 Wire Wire Line
-	6900 3250 6900 3350
-Wire Wire Line
-	6900 3850 6900 4700
-$Comp
-L R-RESCUE-oBeMs_Pulse_PCB R56
-U 1 1 563A6584
-P 7200 3600
-F 0 "R56" V 7280 3600 50  0000 C CNN
-F 1 "120" V 7200 3600 50  0000 C CNN
-F 2 "REInnovationFootprint:TH_Resistor_1" H 7200 3600 60  0001 C CNN
-F 3 "" H 7200 3600 60  0000 C CNN
-F 4 "Value" H 7200 3600 60  0001 C CNN "Description"
-F 5 "Value" H 7200 3600 60  0001 C CNN "Notes"
-F 6 "Value" H 7200 3600 60  0001 C CNN "Manufacturer"
-F 7 "Value" H 7200 3600 60  0001 C CNN "Manufacturer Part No"
-F 8 "Value" H 7200 3600 60  0001 C CNN "Supplier 1"
-F 9 "Value" H 7200 3600 60  0001 C CNN "Supplier 1 Part No"
-F 10 "Value" H 7200 3600 60  0001 C CNN "Supplier 2"
-F 11 "Value" H 7200 3600 60  0001 C CNN "Supplier 2 Part No"
-	1    7200 3600
-	1    0    0    1
-$EndComp
+	6900 3250 6900 4700
 $Comp
 L LED-RESCUE-oBeMs_Pulse_PCB D14
@@
 $EndComp
 Wire Wire Line
-	7200 3250 7200 3350
-Wire Wire Line
-	7200 3850 7200 4800
+	7200 3250 7200 4800
 Wire Wire Line
 	6600 4000 6450 4000

Commit message: Changes for v0001
Multiple PCb changes. 50Pcs ordered
Parts:
- removed Q1: BC546, matts_components:TO92-EBC_large_pad, symbol NPN
- removed U3: TLC555, REInnovationFootprint:DIP-8__300_ELL, symbol TLC555
- added Q1: BC546, matts_components:TO92-PNP_large_pad, symbol Q_NPN_CBE
- added U3: TLC555_8PIN, REInnovationFootprint:DIP-8__300_ELL, symbol TLC555_8PIN
- C4: value 0.1u -> 1u
- C5: value 10n -> 1u
- RV1: footprint matts_components:RV_various_lg_pad -> REInnovationFootprint:RV_various_lg_pad
Changed lines of the file:
@@
 EESchema Schematic File Version 2
-LIBS:oBeMs_Pulse_PCB-rescue
 LIBS:power
 LIBS:device
@@
 Watch Dog Timer
 $Comp
-L TLC555 U3
-U 1 1 5636A483
-P 5100 2700
-F 0 "U3" H 5250 3300 70  0000 C CNN
-F 1 "TLC555" H 5250 2600 70  0000 C CNN
-F 2 "REInnovationFootprint:DIP-8__300_ELL" H 5100 2700 60  0001 C CNN
-F 3 "" H 5100 2700 60  0000 C CNN
-	1    5100 2700
-	1    0    0    -1
-$EndComp
-$Comp
 L C-RESCUE-oBeMs_Pulse_PCB C3
 U 1 1 5636A48A
@@
 P 5750 2900
 F 0 "C5" H 5800 3000 50  0000 L CNN
-F 1 "10n" H 5800 2800 50  0000 L CNN
+F 1 "1u" H 5800 2800 50  0000 L CNN
 F 2 "matts_components:C1_wide_lg_pad_2" H 5750 2900 60  0001 C CNN
 F 3 "" H 5750 2900 60  0000 C CNN
@@
 P 5050 3400
 F 0 "C4" H 5100 3500 50  0000 L CNN
-F 1 "0.1u" H 5100 3300 50  0000 L CNN
+F 1 "1u" H 5100 3300 50  0000 L CNN
 F 2 "matts_components:C1_wide_lg_pad_2" H 5050 3400 60  0001 C CNN
 F 3 "" H 5050 3400 60  0000 C CNN
@@
 $EndComp
 $Comp
-L NPN Q1
-U 1 1 5636A54F
-P 7500 4900
-F 0 "Q1" H 7500 4750 50  0000 R CNN
-F 1 "BC546" H 7500 5050 50  0000 R CNN
-F 2 "matts_components:TO92-EBC_large_pad" H 7500 4900 60  0001 C CNN
-F 3 "http://docs-europe.electrocomponents.com/webdocs/078e/0900766b8078ea72.pdf" H 7500 4900 60  0001 C CNN
-F 4 "NPN. 1A. 80V" H 7500 4900 60  0001 C CNN "Description"
-F 5 "~" H 7500 4900 60  0001 C CNN "Notes"
-F 6 "ON Semiconductor" H 7500 4900 60  0001 C CNN "Manufacturer"
-F 7 "BC639" H 7500 4900 60  0001 C CNN "Manufacturer Part No"
-F 8 "RS" H 7500 4900 60  0001 C CNN "Supplier 1"
-F 9 "545-2276" H 7500 4900 60  0001 C CNN "Supplier 1 Part No"
-F 10 "~" H 7500 4900 60  0001 C CNN "Supplier 2"
-F 11 "~" H 7500 4900 60  0001 C CNN "Supplier 2 Part No"
-F 12 "~" H 7500 4900 60  0001 C CNN "Cost"
-	1    7500 4900
-	1    0    0    -1
-$EndComp
-$Comp
 L R-RESCUE-oBeMs_Pulse_PCB R7
 U 1 1 5636A55D
@@
 	5750 3100 5750 3250
 Wire Wire Line
-	4450 2400 4800 2400
-Wire Wire Line
 	6100 2050 6100 2000
 Wire Wire Line
@@
 Wire Wire Line
 	5750 2300 5700 2300
-Wire Wire Line
-	4650 2500 4800 2500
 Wire Wire Line
 	7600 4150 7600 4050
@@
 +3.3V
 Wire Wire Line
-	4800 2600 4350 2600
-Wire Wire Line
 	5400 850  5750 850
 Wire Wire Line
@@
 F 0 "RV1" H 6100 1150 50  0000 C CNN
 F 1 "500k" H 6100 1250 50  0000 C CNN
-F 2 "matts_components:RV_various_lg_pad" H 6100 1250 60  0001 C CNN
-F 3 "" H 6100 1250 60  0000 C CNN
+F 2 "REInnovationFootprint:RV_various_lg_pad" H 6100 1250 60  0001 C CNN
+F 3 "http://docs-europe.electrocomponents.com/webdocs/002e/0900766b8002e6fe.pdf" H 6100 1250 60  0001 C CNN
+F 4 "~" H 6100 1250 60  0000 C CNN "Notes"
+F 5 "~" H 6100 1250 60  0001 C CNN "Description"
+F 6 "~" H 6100 1250 60  0001 C CNN "Manufacturer"
+F 7 "~" H 6100 1250 60  0001 C CNN "Manufacturer Part No"
+F 8 "~" H 6100 1250 60  0001 C CNN "Supplier 1"
+F 9 "~" H 6100 1250 60  0001 C CNN "Supplier 1 Part No"
+F 10 "~" H 6100 1250 60  0001 C CNN "Supplier 1 Cost"
+F 11 "~" H 6100 1250 60  0001 C CNN "Supplier 2"
+F 12 "~" H 6100 1250 60  0001 C CNN "Supplier 2 Part No"
+F 13 "~" H 6100 1250 60  0001 C CNN "Supplier 2 Cost"
 	1    6100 1250
 	0    -1   -1   0
@@
 Text HLabel 4950 3750 0    60   Input ~ 0
 GND
-Text HLabel 4750 2050 0    60   Input ~ 0
+Text HLabel 4150 2300 0    60   Input ~ 0
 GND
 Text HLabel 5600 3250 0    60   Input ~ 0
@@
 	5050 3750 4950 3750
 Wire Wire Line
-	4750 2050 4800 2050
-Wire Wire Line
-	4800 2050 4800 2300
+	4150 2300 4700 2300
 NoConn ~ 6450 5100
 NoConn ~ 6450 4600
@@
 NoConn ~ 6450 4200
 NoConn ~ 6450 4100
+$Comp
+L Q_NPN_CBE Q1
+U 1 1 5991B6E4
+P 7500 4900
+F 0 "Q1" H 7800 4950 50  0000 R CNN
+F 1 "BC546" H 7950 4850 50  0000 R CNN
+F 2 "matts_components:TO92-PNP_large_pad" H 7700 5000 50  0001 C CNN
+F 3 "" H 7500 4900 50  0000 C CNN
+	1    7500 4900
+	1    0    0    -1
+$EndComp
+$Comp
+L TLC555_8PIN U3
+U 1 1 599187A7
+P 5200 2500
+F 0 "U3" H 5100 2925 50  0000 R CNN
+F 1 "TLC555_8PIN" H 5100 2850 50  0000 R CNN
+F 2 "REInnovationFootprint:DIP-8__300_ELL" H 5250 2250 50  0001 L CNN
+F 3 "" H 5850 1950 50  0000 C CNN
+	1    5200 2500
+	1    0    0    -1
+$EndComp
+Wire Wire Line
+	4650 2500 4700 2500
+Wire Wire Line
+	4700 2600 4350 2600
+Wire Wire Line
+	4450 2400 4700 2400
+Wire Wire Line
+	6100 1500 6100 1400
 $EndSCHEMATC
